File: kicad/KEPR/KEPR.kicad_pcb (KiCad board)
At the start: 2 copper layers, 67.6 x 25.4 mm, 7 parts, among them J10 Conn_02x40_Odd_Even, J2 SODIMM-200, J3 Conn_02x12_Odd_Even, J4 Conn_02x15_Odd_Even, J5 Conn_02x08_Odd_Even, J6 Conn_02x20_Odd_Even, J9 Conn_02x40_Odd_Even

Commit message: Adicionado Footprints, criado a visualização da PCB
Parts:
- moved J10 36.4 mm to (172.5, 216.1)
- moved J2 36.4 mm to (167.0, 84.3)
- moved J3 36.4 mm to (114.0, 111.0)
- moved J4 36.4 mm to (279.9, 84.6)
- moved J6 36.4 mm to (330.1, 213.5)
- moved J9 36.4 mm to (61.5, 216.1)
- moved J5 36.4 mm to (271.5, 134.8)
Changed lines of the file:
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@@
 	)
 	(paper "A3")
+	(title_block
+		(title "UCE Board")
+		(date "2026-01-01")
+		(rev "0.5")
+		(company "Rapport Tecnologia")
+		(comment 1 "Carlos Delfino Carvalho Pinheiro")
+		(comment 2 "consultoria@carlosdelfino.eti.br")
+	)
 	(layers
 		(0 "F.Cu" signal)
@@
 	(footprint "Connector_PinHeader_2.54mm:PinHeader_2x40_P2.54mm_Vertical"
 		(layer "F.Cu")
-		(at 136.52 210.54 90)
+		(at 172.52 216.08 90)
 		(descr "Through hole straight pin header, 2x40, 2.54mm pitch, double rows")
 		(tags "Through hole pin header THT 2x40 2.54mm double row")
@@
 	(footprint "Connector_IDC:IDC-Header_2x25_P2.54mm_Latch6.5mm_Vertical"
 		(layer "F.Cu")
-		(at 78 105.5)
+		(at 114 111.04)
 		(descr "Through hole IDC header, 2x25, 2.54mm pitch, DIN 41651 / IEC 60603-13, double rows, 6.5mm latches, https://docs.google.com/spreadsheets/d/16SsEcesNF15N3Lb4niX7dcUr-NY5_MFPQhobNuNppn4/edit#gid=0")
 		(tags "Through hole vertical IDC header THT 2x25 2.54mm double row")
@@
 	(footprint "Connector_IDC:IDC-Header_2x15-1MP_P2.54mm_Latch_Vertical"
 		(layer "F.Cu")
-		(at 243.94 79.02 90)
+		(at 279.94 84.56 90)
 		(descr "Through hole IDC header, 2x15, 2.54mm pitch, DIN 41651 / IEC 60603-13, double rows latches, mounting holes, https://docs.google.com/spreadsheets/d/16SsEcesNF15N3Lb4niX7dcUr-NY5_MFPQhobNuNppn4/edit#gid=0")
 		(tags "Through hole vertical IDC header THT 2x15 2.54mm double row")
@@
 	(footprint "Connector_PCBEdge:SODIMM-200_2.5V_Card_edge"
 		(layer "F.Cu")
-		(at 131 78.75)
+		(at 167 84.29)
 		(descr "SODIMM 200-pins edge connector, Jedec MO-224 Variation AA compliant (2.5V DDR SDRAM), 0.6mm pitch, https://www.jst-mfg.com/product/pdf/eng/eDM-200P.pdf")
 		(tags "sodimm")
@@
 			(polygon
 				(pts
-					(xy 128.85 66.15) (xy 130.85 66.15) (xy 130.85 60.125) (xy 128.85 60.125)
+					(xy 164.85 71.69) (xy 166.85 71.69) (xy 166.85 65.665) (xy 164.85 65.665)
 				)
 			)
@@
 			(polygon
 				(pts
-					(xy 128.85 77.575) (xy 130.725 77.575) (xy 130.725 80.125) (xy 128.85 80.125)
+					(xy 164.85 83.115) (xy 166.725 83.115) (xy 166.725 85.665) (xy 164.85 85.665)
 				)
 			)
@@
 			(polygon
 				(pts
-					(xy 128.85 80.125) (xy 129.85 80.125) (xy 129.85 66.15) (xy 128.85 66.15)
+					(xy 164.85 85.665) (xy 165.85 85.665) (xy 165.85 71.69) (xy 164.85 71.69)
 				)
 			)
@@
 			(polygon
 				(pts
-					(xy 142.975 77.575) (xy 146.35 77.575) (xy 146.35 80.125) (xy 142.975 80.125)
+					(xy 178.975 83.115) (xy 182.35 83.115) (xy 182.35 85.665) (xy 178.975 85.665)
 				)
 			)
@@
 			(polygon
 				(pts
-					(xy 194.45 66.15) (xy 196.45 66.15) (xy 196.45 60.125) (xy 194.45 60.125)
+					(xy 230.45 71.69) (xy 232.45 71.69) (xy 232.45 65.665) (xy 230.45 65.665)
 				)
 			)
@@
 			(polygon
 				(pts
-					(xy 194.575 77.575) (xy 196.45 77.575) (xy 196.45 80.125) (xy 194.575 80.125)
+					(xy 230.575 83.115) (xy 232.45 83.115) (xy 232.45 85.665) (xy 230.575 85.665)
 				)
 			)
@@
 			(polygon
 				(pts
-					(xy 195.45 80.125) (xy 196.45 80.125) (xy 196.45 66.15) (xy 195.45 66.15)
+					(xy 231.45 85.665) (xy 232.45 85.665) (xy 232.45 71.69) (xy 231.45 71.69)
 				)
 			)
@@
 			(polygon
 				(pts
-					(xy 128.85 62.625) (xy 130.85 62.625) (xy 130.85 60.125) (xy 128.85 60.125)
+					(xy 164.85 68.165) (xy 166.85 68.165) (xy 166.85 65.665) (xy 164.85 65.665)
 				)
 			)
@@
 			(polygon
 				(pts
-					(xy 128.85 80.125) (xy 128.85 79.125) (xy 196.45 79.125) (xy 196.45 80.125)
+					(xy 164.85 85.665) (xy 164.85 84.665) (xy 232.45 84.665) (xy 232.45 85.665)
 				)
 			)
@@
 			(polygon
 				(pts
-					(xy 128.85 80.125) (xy 129.35 80.125) (xy 129.35 62.625) (xy 128.85 62.625)
+					(xy 164.85 85.665) (xy 165.35 85.665) (xy 165.35 68.165) (xy 164.85 68.165)
 				)
 			)
@@
 			(polygon
 				(pts
-					(xy 194.45 62.625) (xy 196.45 62.625) (xy 196.45 60.125) (xy 194.45 60.125)
+					(xy 230.45 68.165) (xy 232.45 68.165) (xy 232.45 65.665) (xy 230.45 65.665)
 				)
 			)
@@
 			(polygon
 				(pts
-					(xy 195.95 80.125) (xy 196.45 80.125) (xy 196.45 62.625) (xy 195.95 62.625)
+					(xy 231.95 85.665) (xy 232.45 85.665) (xy 232.45 68.165) (xy 231.95 68.165)
 				)
 			)
@@
 	(footprint "Connector_IDC:IDC-Header_2x08_P2.54mm_Latch12.0mm_Vertical"
 		(layer "F.Cu")
-		(at 235.46 129.22)
+		(at 271.46 134.76)
 		(descr "Through hole IDC header, 2x08, 2.54mm pitch, DIN 41651 / IEC 60603-13, double rows, 12.0mm latches, https://docs.google.com/spreadsheets/d/16SsEcesNF15N3Lb4niX7dcUr-NY5_MFPQhobNuNppn4/edit#gid=0")
 		(tags "Through hole vertical IDC header THT 2x08 2.54mm double row")
@@
 	(footprint "Connector_PinHeader_2.54mm:PinHeader_2x40_P2.54mm_Vertical"
 		(layer "F.Cu")
-		(at 25.46 210.54 90)
+		(at 61.46 216.08 90)
 		(descr "Through hole straight pin header, 2x40, 2.54mm pitch, double rows")
 		(tags "Through hole pin header THT 2x40 2.54mm double row")
@@
 	(footprint "Connector_PinHeader_2.54mm:PinHeader_2x20_P2.54mm_Vertical"
 		(layer "F.Cu")
-		(at 294.06 208 -90)
+		(at 330.06 213.54 -90)
 		(descr "Through hole straight pin header, 2x20, 2.54mm pitch, double rows")
 		(tags "Through hole pin header THT 2x20 2.54mm double row")
@@
 	)
 	(embedded_fonts no)
+	(embedded_files
+		(file
+			(name "abnt.kicad_wks")
+			(type worksheet)
+			(data |KLUv/WAtCaUUAGZdXSEA1TZqxSYpSnAbOsWn6jgBcMQyc4EzL++4wmTo/39CwQRTAEwAVwAfib/D
+				sXnSvpaTvVHzGxcLF61mdz60Ir9WLFwVbS/Z8kf+BAAgQILey1kpKA2V8dvQNSJJdcbvZb/OIQAC
+				BYxSatVZ+2JbZg8RAIHyI9KEHmg/hLSv2iUmKUr1j/y/v6Z11Z4XaZTBa99z0nP2mzH4Ys+e1AfE
+				4tcuvv32znd4QTh7TfVfH0cM1q4dXj9YPSntz96XFNU+evdBzyP+xwFZpWS5UMRfH+qG0Swht2AY
+				1RBaHVox6YSycRYNo2lkjA1iGlzV1ZNSRYXoBHbSuqyh0S4ct5kGvfD3GjlnUva/DjZpY78Eea7a
+				NCPVq+f3fZNagMBfvAmBAqJeCqtah6qwKKJOi3YTTUK6HjlixqyZSVaRUBiJR5dVOk17cBhmVQdJ
+				NtEim8M6QCt6bztRTapFuq0T33aVhrbfvcMJDCdBuFH93pjxprOTXsWiVQJ/oBFFhhRNSQqSFDLM
+				AXBEpObIdIhoeADgyjYO5AUHII+5zeGUZ8OCCgxpYQqEQHAhLidmCx0AKeQ9n6T/yBrb7V12yDYr
+				OiEXJglxtvK15pFxtmAHCO91fmulXHfWElz75BBUrBctqPwIp/TZhV6iCDIApxHAeXt16x/Kg7DG
+				kiWEXtJRLCUAuZbMBWDdLI5A4osumcUmrV5EsjmvZPcMXsOAYTw4linxEUyETifR+zbQER70Mm3G
+				h/OmhDwS8UnyTSUo/nDK0UuSa6aYZw+3mSUACEI+UaM6ItXawEKAG2ER79AKTrs0yN07DJnJ2GGX
+				ZfKigD5qX0sOMakP3fYKbZusDnmUYtdHdIyXSuldo/AF/MS73bQI2vgwVQ==|
+			)
+			(checksum "9F561F2F5A0DC32E669BBA2695209430")
+		)
+	)
 )

Commit message: Vários ajuste, sendo o mais importante a adição do power rail e iniciado o Wireless module
Parts:
- removed J2: SODIMM-200, Connector_PCBEdge:SODIMM-200_2.5V_Card_edge
- added J11: 10141995-005RLF, Connector_PCBEdge:SODIMM-260_DDR4_H4.0-5.2_OrientationStd_Socket, F.Cu at (189.9, 58.2)
- moved J3 48.0 mm to (66.0, 109.0)
- moved J4 43.7 mm to (266.4, 43.0)
Other:
- board outline removed

Commit message: mais ajustes no power rail inclusive com imagem 3d
Parts:
- added J1: PINHD_1x20_Male, Connector_PinHeader_2.54mm:PinHeader_1x20_P2.54mm_Vertical, F.Cu at (60.7, 209.5)
- added J12: PINHD_1x20_Male, Connector_PinHeader_2.54mm:PinHeader_1x20_P2.54mm_Vertical, F.Cu at (171.7, 209.5)
- added J13: PINHD_1x20_Male, Connector_PinHeader_2.54mm:PinHeader_1x20_P2.54mm_Vertical, F.Cu at (224.0, 209.5)
- added J14: PINHD_2x3_Male, Connector_PinHeader_2.54mm:PinHeader_2x03_P2.54mm_Vertical, F.Cu at (316.8, 201.1)
- added J15: PINHD_1x10_Male, Connector_PinHeader_2.54mm:PinHeader_1x10_P2.54mm_Vertical, F.Cu at (308.0, 209.0)
- added J16: PINHD_1x10_Male, Connector_PinHeader_2.54mm:PinHeader_1x10_P2.54mm_Vertical, F.Cu at (280.9, 209.0)
- added J17: PINHD_1x20_Male, Connector_PinHeader_2.54mm:PinHeader_1x20_P2.54mm_Vertical, F.Cu at (60.7, 205.5)
- added J18: PINHD_1x20_Male, Connector_PinHeader_2.54mm:PinHeader_1x20_P2.54mm_Vertical, F.Cu at (112.9, 205.5)
- added J19: PINHD_1x20_Male, Connector_PinHeader_2.54mm:PinHeader_1x20_P2.54mm_Vertical, F.Cu at (171.8, 205.5)
- added J2: PINHD_1x20_Male, Connector_PinHeader_2.54mm:PinHeader_1x20_P2.54mm_Vertical, F.Cu at (113.0, 209.5)
- added J20: PINHD_1x20_Male, Connector_PinHeader_2.54mm:PinHeader_1x20_P2.54mm_Vertical, F.Cu at (224.0, 205.5)
- added J21: PINHD_1x10_Male, Connector_PinHeader_2.54mm:PinHeader_1x10_P2.54mm_Vertical, F.Cu at (308.0, 205.0)
- added J23: PINHD_1x10_Male, Connector_PinHeader_2.54mm:PinHeader_1x10_P2.54mm_Vertical, F.Cu at (280.9, 205.0)
- added J24: PINHD_2x3_Male, Connector_PinHeader_2.54mm:PinHeader_2x03_P2.54mm_Vertical, F.Cu at (82.5, 201.0)
- added J25: PINHD_2x3_Male, Connector_PinHeader_2.54mm:PinHeader_2x03_P2.54mm_Vertical, F.Cu at (134.9, 201.0)
- added J26: PINHD_2x3_Male, Connector_PinHeader_2.54mm:PinHeader_2x03_P2.54mm_Vertical, F.Cu at (193.4, 201.0)
- added J27: PINHD_2x3_Male, Connector_PinHeader_2.54mm:PinHeader_2x03_P2.54mm_Vertical, F.Cu at (244.5, 201.0)
- added J30: PINHD_2x3_Male, Connector_PinHeader_2.54mm:PinHeader_2x03_P2.54mm_Vertical, F.Cu at (289.3, 201.0)
Connections:
- J11 pad 100: GND -> unconnected-(J11-Pad100)
- J11 pad 128: unconnected-(J11-Pad128) -> GND
- J11 pad 129: unconnected-(J11-Pad129) -> GND
- J11 pad 230: GND -> unconnected-(J11-Pad230)
- J11 pad 231: GND -> unconnected-(J11-Pad231)
- J11 pad 259: unconnected-(J11-Pad259) -> GND
- J11 pad 260: unconnected-(J11-Pad260) -> GND
- J11 pad 99: GND -> unconnected-(J11-Pad99)

Commit message: Adicionado conversores DC-DC e Logo da Rapport
Parts:
- added J22: Barrel_Jack, Barrel Jack:BarrelJack_Horizontal, F.Cu at (71.5, 75.8)
- added PS1: TDN5-2410WISM, TDN 5WISM Series, 5 Watt:CONV_TDN5-2411WISM, F.Cu at (90.2, 73.2)
- added PS2: TDN5-2411WISM, TDN 5WISM Series, 5 Watt:CONV_TDN5-2411WISM, F.Cu at (90.2, 84.3)
- added PS3: TDN_5-2412WISM, TDN 5WISM Series, 5 Watt:CONV_TDN5-2411WISM, F.Cu at (90.2, 95.5)
- added REF**: MountingHole_5.3mm_M5_Pad_Via, Mount Hole:MountingHole_5.3mm_M5_Pad_Via, F.Cu at (353.5, 130.5)
- added REF**: MountingHole_5.3mm_M5_Pad_Via, Mount Hole:MountingHole_5.3mm_M5_Pad_Via, F.Cu at (282.5, 213.0)
- added REF**: MountingHole_5.3mm_M5_Pad_Via, Mount Hole:MountingHole_5.3mm_M5_Pad_Via, F.Cu at (354.0, 32.5)
- added REF**: MountingHole_5.3mm_M5_Pad_Via, Mount Hole:MountingHole_5.3mm_M5_Pad_Via, F.Cu at (287.0, 32.5)
- added REF**: MountingHole_5.3mm_M5_Pad_Via, Mount Hole:MountingHole_5.3mm_M5_Pad_Via, F.Cu at (282.0, 131.0)
- added REF**: MountingHole_5.3mm_M5_Pad_Via, Mount Hole:MountingHole_5.3mm_M5_Pad_Via, F.Cu at (165.3, 32.8)
- added REF**: MountingHole_5.3mm_M5_Pad_Via, Mount Hole:MountingHole_5.3mm_M5_Pad_Via, F.Cu at (354.0, 212.5)
- added REF**: MountingHole_5.3mm_M5_Pad_Via, Mount Hole:MountingHole_5.3mm_M5_Pad_Via, F.Cu at (42.5, 32.5)
- added REF**: MountingHole_5.3mm_M5_Pad_Via, Mount Hole:MountingHole_5.3mm_M5_Pad_Via, F.Cu at (42.0, 212.0)
- added REF**: MountingHole_5.3mm_M5_Pad_Via, Mount Hole:MountingHole_5.3mm_M5_Pad_Via, F.Cu at (162.0, 212.5)
- added REF**: MountingHole_5.3mm_M5_Pad_Via, Mount Hole:MountingHole_5.3mm_M5_Pad_Via, F.Cu at (42.0, 131.0)
- added REF**: MountingHole_5.3mm_M5_Pad_Via, Mount Hole:MountingHole_5.3mm_M5_Pad_Via, F.Cu at (163.0, 131.0)
- moved J5 14.6 mm to (266.5, 121.0)
- moved J15 11.0 mm to (318.9, 209.4)
- moved J16 11.0 mm to (291.9, 209.4)
- moved J21 11.0 mm to (318.9, 205.4)
- moved J14 11.0 mm to (327.8, 201.6)
- moved J30 11.0 mm to (300.3, 201.5)
- moved J6 11.0 mm to (341.0, 214.0)
- moved J23 11.0 mm to (291.8, 205.4)
- moved J24 8.50 mm to (74.0, 201.0)
- moved J1 8.44 mm to (52.3, 209.4)
- moved J17 8.44 mm to (52.3, 205.4)
- moved J18 8.44 mm to (104.4, 205.4)
- moved J2 8.44 mm to (104.5, 209.4)
- moved J9 8.44 mm to (53.0, 216.0)
- moved J25 8.42 mm to (126.5, 201.0)
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Other:
- board outline added: 329.5 x 199.5 mm
- board text added: "https://kepr.rapport.tec.br"

Commit message: Diversos ajustes no Power Rail
Parts:
- removed REF** (x12): MountingHole_5.3mm_M5_Pad_Via, Mount Hole:MountingHole_5.3mm_M5_Pad_Via
- added C1: 4.7nF_Ceramic, Capacitor:C_0805_2012Metric, F.Cu at (104.5, 130.0)
- added C2: 4.7nF_Ceramic, Capacitor:C_0805_2012Metric, F.Cu at (92.0, 127.5)
- added C3: 4.7nF_Ceramic, Capacitor:C_0805_2012Metric, F.Cu at (90.0, 134.0)
- added C4: 4.7nF_Ceramic, Capacitor:C_0805_2012Metric, F.Cu at (100.0, 140.5)
- added D1: BZV55B3V3, Diode_SMD:D_MiniMELF, F.Cu at (101.5, 120.8)
- added G***: LOGO, Logo Rapport:logo_rapport_87x30, F.Cu at (100.0, 41.5)
- added R1: 5.6MR, Resistors SMD:RESC2012X60N, F.Cu at (101.5, 115.5)
- added R2: GMR320HJAAFD5L00, Shunt Rohm:RESC7142X55N, F.Cu at (113.0, 76.0)
- added R3: GMR320HJAAFD5L00, Shunt Rohm:RESC7142X55N, F.Cu at (113.0, 88.5)
- added R4: GMR320HJAAFD5L00, Shunt Rohm:RESC7142X55N, F.Cu at (112.5, 101.0)
- added U2: STM32G484CETx, Package_QFP:LQFP-48_7x7mm_P0.5mm, F.Cu at (97.3, 132.8)
- moved J22 34.9 mm to (47.5, 50.5)
- moved J6 15.2 mm to (343.7, 199.0)
- moved J10 15.2 mm to (175.2, 201.1)
- moved J9 15.2 mm to (55.7, 201.0)
- moved J18 13.6 mm to (106.2, 218.9)
- moved J19 13.6 mm to (173.5, 219.0)
- moved J20 13.6 mm to (225.7, 219.0)
- moved J21 13.6 mm to (320.7, 218.9)
- moved J23 13.6 mm to (293.6, 218.9)
- moved J17 13.6 mm to (54.0, 218.9)
- moved J24 8.19 mm to (75.7, 209.0)
- moved J25 8.14 mm to (128.0, 209.0)
- moved J30 7.89 mm to (302.5, 209.0)
- moved J14 7.80 mm to (330.0, 209.0)
- moved J26 7.77 mm to (195.5, 208.5)
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Connections:
- net /Power Rails/External Power Rails/UCE_MCU_VCTL_12v renamed /Power/External Power Rails/UCE_MCU_VCTL_12v
- net /Power Rails/External Power Rails/UCE_MCU_VCTL_3v3 renamed /Power/External Power Rails/UCE_MCU_VCTL_3v3
- net /Power Rails/External Power Rails/UCE_MCU_VCTL_5V renamed /Power/External Power Rails/UCE_MCU_VCTL_5V
- PS1 pad 7: +3.3V -> /Power/External Power Rails/+3.3v Shunt
- PS2 pad 7: +5V -> /Power/External Power Rails/+5v Shunt
- PS3 pad 7: +12V -> /Power/External Power Rails/12v Shunt
Routing:
- net GND: track 0.00 -> 1828.8 mm, vias 0 -> 36
- net +24V: track 0.00 -> 109.8 mm
- net Net-(J2-Pad1): track 0.00 -> 59.8 mm
- net Net-(J1-Pad1): track 0.00 -> 59.6 mm
- net Net-(J13-Pad1): track 0.00 -> 58.9 mm
- net /UCE board/VDD_Z_MCU_CTL_3v3: track 0.00 -> 54.9 mm
- net +3.3V: track 0.00 -> 44.4 mm, vias 0 -> 2
- net Net-(J14-Pad1): track 0.00 -> 34.3 mm
- net Net-(J16-Pad1): track 0.00 -> 26.7 mm
- net Net-(J12-Pad1): track 0.00 -> 11.9 mm
- net (no net): track 0.00 -> 0.77 mm

Commit message: Mais ajustes no roteamento
Parts:
- moved R4 2.50 mm to (112.5, 98.5)
- moved R3 1.54 mm to (112.7, 87.0)
Connections:
- PS1 pad 7: /Power/External Power Rails/+3.3v Shunt -> +3v3 Shunt
- PS2 pad 7: /Power/External Power Rails/+5v Shunt -> +5v Shunt
- PS3 pad 7: /Power/External Power Rails/12v Shunt -> +12v Shunt
- R2 pad 1: /UCE board/+3.3v Shunt -> +3v3 Shunt
- R3 pad 1: /UCE board/+5v Shunt -> +5v Shunt
- R4 pad 1: /UCE board/12v Shunt -> +12v Shunt
- U2 pad 11: unconnected-(U2-PA3-Pad11) -> +3v3 Shunt
- U2 pad 13: unconnected-(U2-PA5-Pad13) -> +5v Shunt
- U2 pad 15: unconnected-(U2-PA7-Pad15) -> +5V
- U2 pad 16: unconnected-(U2-PB0-Pad16) -> +12V
- U2 pad 18: unconnected-(U2-PB2-Pad18) -> +12v Shunt
- U2 pad 9: unconnected-(U2-PA1-Pad9) -> +3.3V
Routing:
- net +5v Shunt: track 0.00 -> 96.1 mm, vias 0 -> 2
- net +3v3 Shunt: track 0.00 -> 91.2 mm, vias 0 -> 2
- net +5V: track 0.00 -> 76.3 mm
- net +12V: track 0.00 -> 63.2 mm
- net +12v Shunt: track 0.00 -> 54.7 mm, vias 0 -> 2
- net +3.3V: track 44.4 -> 87.3 mm, vias 2 -> 4
- net /UCE board/VDD_Z_MCU_CTL_3v3: track 54.9 -> 64.5 mm, vias 0 -> 9
- net GND: track 1828.8 -> 1835.1 mm, vias 36 -> 44

Commit message: Ajustes no Power Rail, entre outros ajustes.
Parts:
- removed J13, J18, J2, J20: PINHD_1x20_Male, Connector_PinHeader_2.54mm:PinHeader_1x20_P2.54mm_Vertical
- removed J14, J25, J27: PINHD_2x3_Male, Connector_PinHeader_2.54mm:PinHeader_2x03_P2.54mm_Vertical
- removed J15, J21: PINHD_1x10_Male, Connector_PinHeader_2.54mm:PinHeader_1x10_P2.54mm_Vertical
- R2: value GMR320HJAAFD5L00 -> GMR320HJAAFM5L00
- R3: value GMR320HJAAFD5L00 -> GMR320HJAAFS5L00
- R4: value GMR320HJAAFD5L00 -> GMR320HJAAFE5L00
Connections:
- net Net-(J1-Pad1) renamed /Power/External Power Rails/Vout_external_1
- net Net-(J12-Pad1) renamed /Power/External Power Rails/Vout_external_2
- net Net-(J16-Pad1) renamed /Power/External Power Rails/Vout_external_3
- J11 pad 100: unconnected-(J11-Pad100) -> I2C_SDA_MCU_CTL
- J11 pad 99: unconnected-(J11-Pad99) -> I2C_SCL_MCU_CTL
- U2 pad 37: unconnected-(U2-PA13-Pad37) -> I2C_SDA_MCU_CTL
- U2 pad 38: unconnected-(U2-PA14-Pad38) -> I2C_SCL_MCU_CTL
- U2 pad 9: +3.3V -> /UCE board/+3.3v Shunt Out
Routing:
- net GND: track 1835.1 -> 1980.2 mm, vias 44 -> 46
- net I2C_SDA_MCU_CTL: track 0.00 -> 125.5 mm, vias 0 -> 2
- net I2C_SCL_MCU_CTL: track 0.00 -> 112.2 mm, vias 0 -> 4
- net Net-(J2-Pad1): track 59.8 -> 0.00 mm
- net Net-(J13-Pad1): track 58.9 -> 0.00 mm
- net Net-(J14-Pad1): track 34.3 -> 0.00 mm
- net MCU_RST_N: track 0.00 -> 11.1 mm
- net I2C0_SCL: track 0.00 -> 10.7 mm
- net I2C2_SCL: track 0.00 -> 9.95 mm
- net UART1_TX: track 0.00 -> 9.65 mm
- net VIO_BANK2: track 0.00 -> 8.87 mm, vias 0 -> 1
- net VCC_IN: track 0.00 -> 7.34 mm
- net VREF_IO: track 0.00 -> 5.87 mm, vias 0 -> 1
- net PWR_GOOD: track 0.00 -> 4.24 mm
- net VIO_BANK0: track 0.00 -> 3.50 mm
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
Commit message: Adicionado holder para bateria.
Parts:
- added BT1: Battery_Cell, Battery:BatteryHolder_Multicomp_BC-2001_1x2032, F.Cu at (91.8, 165.0)
Connections:
- U2 pad 1: unconnected-(U2-VBAT-Pad1) -> Net-(BT1-+)
Routing:
- net Net-(BT1-+): track 0.00 -> 59.8 mm, vias 0 -> 2
- net GND: track 1980.2 -> 2008.0 mm, vias 46 -> 47
- net /UCE board/VDD_Z_MCU_CTL_3v3: track 64.5 -> 65.4 mm
