File: kicad/KEPR/KEPR.kicad_pcb (KiCad board)
At the start: 4 copper layers, 329.5 x 199.5 mm, 36 parts, among them IC1 ACS37041KLHBLT-010B3, IC2 ACS37041KLHBLT-010B3, IC3 ACS37041KLHBLT-010B3, J1 PINHD_1x20_Male, J10 Conn_02x40_Odd_Even, J11 10141995-005RLF, J12 PINHD_1x20_Male, J13 PINHD_2x2_Male, J16 PINHD_1x10_Male, J17 PINHD_1x20_Male, J19 PINHD_1x20_Male, J22 Barrel_Jack, J23 PINHD_1x10_Male, J24 PINHD_2x2_Male, J26 PINHD_2x3_Male, J3 Conn_02x12_Odd_Even, J30 PINHD_2x2_Male, J4 Conn_02x15_Odd_Even, J5 Conn_02x08_Odd_Even, J6 Conn_02x20_Odd_Even, J9 Conn_02x40_Odd_Even, U1 REF193, U2 STM32G484CETx, U3 AMS1117-3.3, U4 AMS1117-1.8

Commit message: Ajustando trilhas
Parts:
- moved J30 1.54 mm to (345.5, 213.0)
Connections:
- J10 pad 59: VIO_BANK0 -> unconnected-(J10-Pin_59-Pad59)
- J10 pad 60: VIO_BANK1 -> unconnected-(J10-Pin_60-Pad60)
- J10 pad 61: VIO_BANK2 -> unconnected-(J10-Pin_61-Pad61)
- J10 pad 62: VIO_BANK3 -> unconnected-(J10-Pin_62-Pad62)
- J10 pad 66: RESERVED -> unconnected-(J10-Pin_66-Pad66)
- J24 pad 1: unconnected-(J24-Pad1) -> /Power/Power Rails/Vout_external_1
- J24 pad 2: unconnected-(J24-Pad2) -> +5V
- J24 pad 3: unconnected-(J24-Pad3) -> /Power/Power Rails/Vout_external_1
- J24 pad 4: unconnected-(J24-Pad4) -> +3.3V
- J30 pad 1: unconnected-(J30-Pad1) -> /Power/Power Rails/Vout_external_3
- J30 pad 2: unconnected-(J30-Pad2) -> +5V
- J30 pad 3: unconnected-(J30-Pad3) -> /Power/Power Rails/Vout_external_3
- J30 pad 4: unconnected-(J30-Pad4) -> +3.3V
Routing:
- net +5V: track 375.2 -> 519.1 mm, vias 7 -> 11
- net I2S_DOUT: track 0.00 -> 133.6 mm, vias 0 -> 1
- net I2S_BCLK: track 16.4 -> 122.0 mm
- net I2C1_SCL: track 63.8 -> 168.4 mm, vias 1 -> 2
- net I2S_MCLK: track 18.6 -> 122.3 mm
- net VCC_IN: track 227.3 -> 317.9 mm, vias 2 -> 3
- net UART1_RX: track 169.3 -> 103.3 mm
- net UART3_RX: track 250.6 -> 187.8 mm, vias 3 -> 5
- net +3.3V: track 652.9 -> 590.4 mm, vias 13 -> 8
- net MCU_EN: track 43.5 -> 95.7 mm
- net unconnected-(J6-Pin_15-Pad15): track 51.7 -> 0.00 mm
- net MCU_BOOT1: track 41.7 -> 93.3 mm
- net VREF_IO: track 74.7 -> 105.0 mm, vias 2 -> 5
- net +1v8: track 118.2 -> 146.8 mm
- net I2S_DIN: track 0.00 -> 28.1 mm, vias 0 -> 1
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