File: kicad/KEPR/KEPR.kicad_pcb (KiCad board)
At the start: 4 copper layers, 329.5 x 199.5 mm, 36 parts, among them IC1 ACS37041KLHBLT-010B3, IC2 ACS37041KLHBLT-010B3, IC3 ACS37041KLHBLT-010B3, J1 PINHD_1x20_Male, J10 Conn_02x40_Odd_Even, J11 10141995-005RLF, J12 PINHD_1x20_Male, J13 PINHD_2x2_Male, J16 PINHD_1x10_Male, J17 PINHD_1x20_Male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

Commit message: mais ajustes de trilha.
Connections:
- J10 pad 31: RESERVED -> unconnected-(J10-Pin_31-Pad31)
- J10 pad 32: RESERVED -> unconnected-(J10-Pin_32-Pad32)
- J11 pad 194: RESERVED -> unconnected-(J11-Pad194)
- J11 pad 201: VIO_BANK1 -> unconnected-(J11-Pad201)
- J11 pad 202: VIO_BANK3 -> unconnected-(J11-Pad202)
- J11 pad 63: RESERVED -> unconnected-(J11-Pad63)
- J3 pad 16: NET_D2_EVEN -> NET_D3_EVEN
Routing:
- net NET_D0_EVEN: track 0.00 -> 180.9 mm, vias 0 -> 2
- net NET_CTL0_ODD: track 0.00 -> 172.0 mm, vias 0 -> 2
- net MDIO: track 0.00 -> 170.0 mm, vias 0 -> 2
- net NET_D2_EVEN: track 0.00 -> 167.6 mm, vias 0 -> 2
- net NET_CLK_ODD: track 0.00 -> 146.8 mm
- net UART0_RTS: track 5.52 -> 152.1 mm, vias 0 -> 1
- net AOUT0: track 9.91 -> 137.4 mm, vias 0 -> 4
- net UART0_DSR: track 34.3 -> 154.2 mm, vias 0 -> 2
- net VREF_IO: track 105.0 -> 221.7 mm, vias 5 -> 10
- net UART3_TX: track 42.5 -> 153.9 mm
- net MCU_RST_N: track 100.9 -> 208.3 mm
- net UART0_DCD: track 6.00 -> 106.6 mm
- net VCC_IN: track 317.9 -> 225.6 mm, vias 3 -> 5
- net UART0_CTS: track 8.68 -> 97.8 mm, vias 0 -> 2
- net +3.3V: track 590.4 -> 667.1 mm
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
Commit message: Mais trilhas e vias lançadas
Parts:
- added J7: Conn_02x08_Odd_Even, Connector_PinHeader_2.00mm:PinHeader_2x08_P2.00mm_Vertical, F.Cu at (248.5, 186.5)
- added J8: Conn_01x08_Pin, Connector_PinHeader_2.00mm:PinHeader_1x08_P2.00mm_Vertical, F.Cu at (248.5, 181.5)
- moved J13 4.06 mm to (257.5, 190.5), turned to -90 degrees
Connections:
- J11 pad 200: VREF_IO -> unconnected-(J11-Pad200)
- J11 pad 226: VREF_IO -> unconnected-(J11-Pad226)
- J11 pad 229: PWR_GOOD -> unconnected-(J11-Pad229)
- J11 pad 69: VREF_IO -> unconnected-(J11-Pad69)
- J11 pad 95: VREF_IO -> unconnected-(J11-Pad95)
- J11 pad 98: PWR_GOOD -> unconnected-(J11-Pad98)
- J13 pad 1: unconnected-(J13-Pad1) -> Net-(J7-Pin_10)
- J13 pad 2: unconnected-(J13-Pad2) -> +3.3V
- J13 pad 3: unconnected-(J13-Pad3) -> Net-(J7-Pin_10)
- J13 pad 4: unconnected-(J13-Pad4) -> +5V
Routing:
- net SPI0_CS2: track 0.00 -> 170.6 mm, vias 0 -> 5
- net SPI0_MOSI: track 0.00 -> 169.9 mm, vias 0 -> 4
- net SPI0_MISO: track 0.00 -> 164.6 mm, vias 0 -> 2
- net SPI0_CS0: track 0.00 -> 163.9 mm, vias 0 -> 4
- net UART2_TX: track 33.7 -> 187.7 mm, vias 1 -> 3
- net SPI1_SCK: track 0.00 -> 153.1 mm, vias 0 -> 5
- net GPIO0: track 12.6 -> 154.0 mm, vias 0 -> 2
- net SPI0_CS1: track 16.6 -> 152.6 mm, vias 0 -> 2
- net I2C1_SDA: track 39.6 -> 170.2 mm, vias 0 -> 2
- net SPI1_MISO: track 16.0 -> 146.1 mm, vias 0 -> 3
- net GPIO2: track 13.2 -> 141.3 mm, vias 0 -> 4
- net UART1_TX: track 61.8 -> 189.0 mm, vias 1 -> 2
- net UART2_RX: track 35.2 -> 157.7 mm, vias 0 -> 4
- net SPI1_CS1: track 0.00 -> 121.9 mm, vias 0 -> 1
- net I2C0_SCL: track 82.8 -> 202.4 mm, vias 2 -> 3
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