File: kicad/KEPR/MCU_Board_STM32N6.kicad_sch (KiCad schematic)
At the start: 0 parts

Commit message: Adicionado a primeira versão da MCU Board, inicado com STM32N6
Parts:
- added J2: 10141995-005RLF, SODIMM DDR4 EDGE 260 pins:SODIMM_DDR4_EDGE, symbol 10141995-005RLF:10141995-005RLF
Connections:
- new net AIN0: J2.44
- new net AIN1: J2.45
- new net AIN2: J2.46
- new net AIN3: J2.47
- new net AIN4: J2.175
- new net AIN5: J2.176
- new net AIN6: J2.177
- new net AIN7: J2.178
- new net AOUT0: J2.48
- new net AOUT1: J2.179
- new net CLOCK_0: J2.205, J2.74
- new net DBG_RESET_N: J2.86
- new net DBG_SWCLK: J2.214
- new net DBG_SWDIO: J2.83
- new net DBG_TCK: J2.84
- new net DBG_TDI: J2.85
- new net DBG_TDO: J2.216
- new net DBG_TMS: J2.215
- new net DBG_UART_RX: J2.218
- new net DBG_UART_TX: J2.87
- new net DBG_VREF: J2.217
- new net GND: J2.1, J2.10, J2.11, J2.128, J2.129, J2.132, J2.133, J2.141, J2.142, J2.143, J2.155, J2.182, J2.195, J2.196, J2.2, J2.203, J2.204, J2.221, J2.222, J2.259, J2.260, J2.64, J2.65, J2.72, J2.73, J2.90, J2.91
- new net GPIO0: J2.31
- new net GPIO1: J2.32
- new net GPIO10: J2.164
- new net GPIO11: J2.165
- new net GPIO12: J2.166
- new net GPIO13: J2.167
- new net GPIO14: J2.168
- new net GPIO15: J2.169
- new net GPIO2: J2.33
- new net GPIO3: J2.34
- new net GPIO4: J2.35
- new net GPIO5: J2.36
- new net GPIO6: J2.37
- new net GPIO7: J2.38
- new net GPIO8: J2.162
- new net GPIO9: J2.163
- new net I2C0_SCL: J2.15
- new net I2C0_SDA: J2.146
- new net I2C1_SCL: J2.16
- new net I2C1_SDA: J2.147
- new net I2C2_SCL: J2.17
- new net I2C2_SDA: J2.148
- new net I2C_SCL_MCU_CTL: J2.99
- new net I2C_SDA_MCU_CTL: J2.100
- new net I2S_BCLK: J2.49
- new net I2S_DIN: J2.181
- new net I2S_DOUT: J2.50
- new net I2S_LRCLK: J2.180
- new net I2S_MCLK: J2.51
- new net IR_RX_IN: J2.43
- new net IR_TX_OUT: J2.174
- new net MCU_BOOT0: J2.14
- new net MCU_BOOT1: J2.145
- new net MCU_EN: J2.144
- new net MCU_RST_N: J2.13
- new net MDIO: J2.59
- new net MOD_PRESENT_N: J2.88
- new net MOD_TYPE0: J2.219
- new net MOD_TYPE1: J2.89
- new net MOD_TYPE2: J2.220
- new net NET_INT_N: J2.54
- new net NET_RST_N: J2.185
- new net NET_SPI_CS: J2.184
- new net NET_SPI_MISO: J2.53
- new net NET_SPI_MOSI: J2.183
- new net NET_SPI_SCK: J2.52
- new net PHY_RST_N: J2.190
- new net PWM0: J2.39
- new net PWM1: J2.40
- new net PWM2: J2.41
- new net PWM3: J2.42
- new net PWM4: J2.170
- new net PWM5: J2.171
- new net PWM6: J2.172
- new net PWM7: J2.173
- new net PWR_GOOD: J2.140, J2.229, J2.9, J2.98
- new net RESERVED: J2.194, J2.206, J2.207, J2.208, J2.209, J2.210, J2.211, J2.212, J2.213, J2.63, J2.75, J2.76, J2.77, J2.78, J2.79, J2.80, J2.81, J2.82
- new net RMII_CRS_DV: J2.188
- new net RMII_REFCLK: J2.58
- new net RMII_RXD0: J2.56
- new net RMII_RXD1: J2.187
- new net RMII_TXD0: J2.55
- new net RMII_TXD1: J2.186
- new net RMII_TXEN: J2.57
- new net SDIO_CLK: J2.60
- new net SDIO_CMD: J2.191
- new net SDIO_D0: J2.61
- new net SDIO_D1: J2.192
- new net SDIO_D2: J2.62
- new net SDIO_D3: J2.193
- new net SPI0_CS0: J2.157
- new net SPI0_CS1: J2.27
- new net SPI0_CS2: J2.158
- new net SPI0_MISO: J2.26
- new net SPI0_MOSI: J2.156
- new net SPI0_SCK: J2.25
- new net SPI1_CS0: J2.160
- new net SPI1_CS1: J2.30
- new net SPI1_CS2: J2.161
- new net SPI1_MISO: J2.29
- new net SPI1_MOSI: J2.159
- new net SPI1_SCK: J2.28
- new net UART0_CTS: J2.22
- new net UART0_DCD: J2.154
- new net UART0_DSR: J2.23
- new net UART0_RI: J2.24
- new net UART0_RTS: J2.153
- new net UART0_RX: J2.149
- new net UART0_TX: J2.18
- new net UART1_RX: J2.150
- new net UART1_TX: J2.19
- new net UART2_RX: J2.151
- new net UART2_TX: J2.20
- new net UART3_RX: J2.152
- new net UART3_TX: J2.21
- new net VCC_1V8: J2.135, J2.199, J2.224, J2.5, J2.68, J2.94
- new net VCC_3V3: J2.136, J2.198, J2.225, J2.4, J2.67, J2.93
- new net VCC_5V: J2.134, J2.197, J2.223, J2.3, J2.66, J2.92
- new net VCC_IN: J2.12
- new net VIO_BANK0: J2.7, J2.70, J2.96
- new net VIO_BANK1: J2.138, J2.201, J2.227
- new net VIO_BANK2: J2.71, J2.8, J2.97
- new net VIO_BANK3: J2.139, J2.202, J2.228
- new net VREF_IO: J2.137, J2.200, J2.226, J2.6, J2.69, J2.95
- new net sMDC: J2.189
Other:
- removed sheet BUSes
- removed sheet MCU Boards
- removed sheet Power
- removed sheet UCE board
- title: KEPR -> (none)
