File: kicad/KEPR/UCE_Bus.kicad_sch (KiCad schematic)
At the start: 1 part, among them J1 SODIMM-200

Commit message: Ajustado a hierarquia de esquemáticos para melhorar o planejamento da placa.
Parts:
- renumbered J1 to J2
Connections:
- net AIN0: no longer J2.87
- net AIN1: no longer J2.89
- net AIN2: no longer J2.91
- net AIN3: no longer J2.93
- net AIN4: no longer J2.88
- net AIN5: no longer J2.90
- net AIN6: no longer J2.92
- net AIN7: no longer J2.94
- net AOUT0: no longer J2.95
- net AOUT1: no longer J2.96
- net CLOCK_0: no longer J2.147, J2.148
- net DBG_RESET_N: no longer J2.171
- net DBG_SWCLK: no longer J2.166
- net DBG_SWDIO: no longer J2.165
- net DBG_TCK: no longer J2.167
- net DBG_TDI: no longer J2.169
- net DBG_TDO: no longer J2.170
- net DBG_TMS: no longer J2.168
- net DBG_UART_RX: no longer J2.174
- net DBG_UART_TX: no longer J2.173
- net DBG_VREF: no longer J2.172
- net GND: now also J2.2, J2.27, J2.28, J2.29, J2.30; no longer J2.102, J2.127, J2.128, J2.129, J2.130, J2.143, J2.144, J2.145, J2.146, J2.179, J2.180, J2.181, J2.182, J2.197, J2.198, J2.199, J2.200, J2.48
- net GPIO0: no longer J2.61
- net GPIO1: no longer J2.63
- net GPIO10: no longer J2.66
- net GPIO11: no longer J2.68
- net GPIO12: no longer J2.70
- net GPIO13: no longer J2.72
- net GPIO14: no longer J2.74
- net GPIO15: no longer J2.76
- net GPIO2: no longer J2.65
- net GPIO3: no longer J2.67
- net GPIO4: no longer J2.69
- net GPIO5: no longer J2.71
- net GPIO6: no longer J2.73
- net GPIO7: no longer J2.75
- net GPIO8: no longer J2.62
- net GPIO9: no longer J2.64
- net I2S_BCLK: no longer J2.97
- net I2S_DIN: no longer J2.100
- net I2S_DOUT: no longer J2.99
- net I2S_LRCLK: no longer J2.98
- net I2S_MCLK: now also J2.1; no longer J2.101
- net IR_RX_IN: no longer J2.85
- net IR_TX_OUT: no longer J2.86
- net MDIO: now also J2.17; no longer J2.117
- net MOD_PRESENT_N: no longer J2.175
- net MOD_TYPE0: no longer J2.176
- net MOD_TYPE1: no longer J2.177
- net MOD_TYPE2: no longer J2.178
- net NET_INT_N: now also J2.7; no longer J2.107
- net NET_RST_N: now also J2.8; no longer J2.108
- net NET_SPI_CS: now also J2.6; no longer J2.106
- net NET_SPI_MISO: now also J2.5; no longer J2.105
- net NET_SPI_MOSI: now also J2.4; no longer J2.104
- net NET_SPI_SCK: now also J2.3; no longer J2.103
- net PHY_RST_N: now also J2.18; no longer J2.118
- net PWM0: no longer J2.77
- net PWM1: no longer J2.79
- net PWM2: no longer J2.81
- net PWM3: no longer J2.83
- net PWM4: no longer J2.78
- net PWM5: no longer J2.80
- net PWM6: no longer J2.82
- net PWM7: no longer J2.84
- net PWR_GOOD: no longer J2.195, J2.196
- net RESERVED: now also J2.25, J2.26; no longer J2.125, J2.126, J2.149, J2.150, J2.151, J2.152, J2.153, J2.154, J2.155, J2.156, J2.157, J2.158, J2.159, J2.160, J2.161, J2.162, J2.163, J2.164
- net RMII_CRS_DV: now also J2.14; no longer J2.114
- net RMII_REFCLK: now also J2.15; no longer J2.115
- net RMII_RXD0: now also J2.11; no longer J2.111
- net RMII_RXD1: now also J2.12; no longer J2.112
- net RMII_TXD0: now also J2.9; no longer J2.109
- net RMII_TXD1: now also J2.10; no longer J2.110
- net RMII_TXEN: now also J2.13; no longer J2.113
- net SDIO_CLK: now also J2.19; no longer J2.119
- net SDIO_CMD: now also J2.20; no longer J2.120
- net SDIO_D0: now also J2.21; no longer J2.121
- net SDIO_D1: now also J2.22; no longer J2.122
- net SDIO_D2: now also J2.23; no longer J2.123
- net SDIO_D3: now also J2.24; no longer J2.124
- net SPI0_CS0: no longer J2.52
- net SPI0_CS1: no longer J2.53
- net SPI0_CS2: no longer J2.54
- net SPI0_MISO: no longer J2.51
- net SPI0_MOSI: no longer J2.50
- net SPI0_SCK: no longer J2.49
- net SPI1_CS0: no longer J2.58
- net SPI1_CS1: no longer J2.59
- net SPI1_CS2: no longer J2.60
- net SPI1_MISO: no longer J2.57
- net SPI1_MOSI: no longer J2.56
- net SPI1_SCK: no longer J2.55
- net UART0_CTS: no longer J2.43
- net UART0_DCD: no longer J2.46
- net UART0_DSR: no longer J2.45
- net UART0_RI: no longer J2.47
- net UART0_RTS: no longer J2.44
- net UART3_RX: no longer J2.42
- net UART3_TX: no longer J2.41
- net VCC_1V8: now also J2.35, J2.36; no longer J2.135, J2.136, J2.186, J2.187
- net VCC_3V3: now also J2.33, J2.34; no longer J2.133, J2.134, J2.185, J2.188
- net VCC_5V: now also J2.31, J2.32; no longer J2.131, J2.132, J2.183, J2.184
- net VIO_BANK0: now also J2.39; no longer J2.139, J2.191
- net VIO_BANK1: now also J2.40; no longer J2.140, J2.192
- net VIO_BANK2: no longer J2.141, J2.193
- net VIO_BANK3: no longer J2.142, J2.194
- net VREF_IO: now also J2.37, J2.38; no longer J2.137, J2.138, J2.189, J2.190
- net sMDC: now also J2.16; no longer J2.116
Changed lines of the file:
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@@
 		(title "UCE Bus (SO-DIMM 200)")
 		(date "2025-12-31")
-		(rev "0.4")
+		(rev "0.5")
 		(company "Rapport Tecnologia")
 	)
@@
 		)
 		(instances
-			(project ""
-				(path "/9d5cdb25-ec8b-4f33-9f87-5d2f7e7c8b1a"
+			(project "KEPR"
+				(path "/5d9e1dfb-5ec5-4e06-bbdb-9cbfa1c0b9f1/0260e008-78ae-4c2c-85f8-b31739d2ea08/f6e289d8-1e57-42c9-86d8-5b4c62dbd3c6"
 					(reference "J1")
 					(unit 1)
@@
 		(lib_id "Connector:SODIMM-200")
 		(at 167.64 147.32 0)
-		(unit 2)
+		(unit 1)
 		(exclude_from_sim no)
 		(in_bom yes)
@@
 		(dnp no)
 		(fields_autoplaced yes)
-		(property "Reference" "J1"
+		(property "Reference" "J2"
 			(at 167.64 41.91 0)
 			(effects
@@
 		)
 		(instances
-			(project ""
-				(path "/9d5cdb25-ec8b-4f33-9f87-5d2f7e7c8b1a"
-					(reference "J1")
-					(unit 2)
+			(project "KEPR"
+				(path "/5d9e1dfb-5ec5-4e06-bbdb-9cbfa1c0b9f1/0260e008-78ae-4c2c-85f8-b31739d2ea08/f6e289d8-1e57-42c9-86d8-5b4c62dbd3c6"
+					(reference "J2")
+					(unit 1)
 				)
 			)
 		)
 	)
-	(sheet_instances
-		(path "/"
-			(page "A0")
-		)
-	)
-	(embedded_fonts no)
 )

Commit message: Definido os demais buses, criado folha do carimbo, versão 0.5
Connections:
- net AIN0: now also J2.87
- net AIN1: now also J2.89
- net AIN2: now also J2.91
- net AIN3: now also J2.93
- net AIN4: now also J2.88
- net AIN5: now also J2.90
- net AIN6: now also J2.92
- net AIN7: now also J2.94
- net AOUT0: now also J2.95
- net AOUT1: now also J2.96
- net CLOCK_0: now also J2.147, J2.148
- net DBG_RESET_N: now also J2.171
- net DBG_SWCLK: now also J2.166
- net DBG_SWDIO: now also J2.165
- net DBG_TCK: now also J2.167
- net DBG_TDI: now also J2.169
- net DBG_TDO: now also J2.170
- net DBG_TMS: now also J2.168
- net DBG_UART_RX: now also J2.174
- net DBG_UART_TX: now also J2.173
- net DBG_VREF: now also J2.172
- net GND: now also J2.102, J2.127, J2.128, J2.129, J2.130, J2.143, J2.144, J2.145, J2.146, J2.179, J2.180, J2.181, J2.182, J2.197, J2.198, J2.199, J2.200, J2.48; no longer J2.2, J2.27, J2.28, J2.29, J2.30
- net GPIO0: now also J2.61
- net GPIO1: now also J2.63
- net GPIO10: now also J2.66
- net GPIO11: now also J2.68
- net GPIO12: now also J2.70
- net GPIO13: now also J2.72
- net GPIO14: now also J2.74
- net GPIO15: now also J2.76
- net GPIO2: now also J2.65
- net GPIO3: now also J2.67
- net GPIO4: now also J2.69
- net GPIO5: now also J2.71
- net GPIO6: now also J2.73
- net GPIO7: now also J2.75
- net GPIO8: now also J2.62
- net GPIO9: now also J2.64
- net I2S_BCLK: now also J2.97
- net I2S_DIN: now also J2.100
- net I2S_DOUT: now also J2.99
- net I2S_LRCLK: now also J2.98
- net I2S_MCLK: now also J2.101; no longer J2.1
- net IR_RX_IN: now also J2.85
- net IR_TX_OUT: now also J2.86
- net MDIO: now also J2.117; no longer J2.17
- net MOD_PRESENT_N: now also J2.175
- net MOD_TYPE0: now also J2.176
- net MOD_TYPE1: now also J2.177
- net MOD_TYPE2: now also J2.178
- net NET_INT_N: now also J2.107; no longer J2.7
- net NET_RST_N: now also J2.108; no longer J2.8
- net NET_SPI_CS: now also J2.106; no longer J2.6
- net NET_SPI_MISO: now also J2.105; no longer J2.5
- net NET_SPI_MOSI: now also J2.104; no longer J2.4
- net NET_SPI_SCK: now also J2.103; no longer J2.3
- net PHY_RST_N: now also J2.118; no longer J2.18
- net PWM0: now also J2.77
- net PWM1: now also J2.79
- net PWM2: now also J2.81
- net PWM3: now also J2.83
- net PWM4: now also J2.78
- net PWM5: now also J2.80
- net PWM6: now also J2.82
- net PWM7: now also J2.84
- net PWR_GOOD: now also J2.195, J2.196
- net RESERVED: now also J2.125, J2.126, J2.149, J2.150, J2.151, J2.152, J2.153, J2.154, J2.155, J2.156, J2.157, J2.158, J2.159, J2.160, J2.161, J2.162, J2.163, J2.164; no longer J2.25, J2.26
- net RMII_CRS_DV: now also J2.114; no longer J2.14
- net RMII_REFCLK: now also J2.115; no longer J2.15
- net RMII_RXD0: now also J2.111; no longer J2.11
- net RMII_RXD1: now also J2.112; no longer J2.12
- net RMII_TXD0: now also J2.109; no longer J2.9
- net RMII_TXD1: now also J2.110; no longer J2.10
- net RMII_TXEN: now also J2.113; no longer J2.13
- net SDIO_CLK: now also J2.119; no longer J2.19
- net SDIO_CMD: now also J2.120; no longer J2.20
- net SDIO_D0: now also J2.121; no longer J2.21
- net SDIO_D1: now also J2.122; no longer J2.22
- net SDIO_D2: now also J2.123; no longer J2.23
- net SDIO_D3: now also J2.124; no longer J2.24
- net SPI0_CS0: now also J2.52
- net SPI0_CS1: now also J2.53
- net SPI0_CS2: now also J2.54
- net SPI0_MISO: now also J2.51
- net SPI0_MOSI: now also J2.50
- net SPI0_SCK: now also J2.49
- net SPI1_CS0: now also J2.58
- net SPI1_CS1: now also J2.59
- net SPI1_CS2: now also J2.60
- net SPI1_MISO: now also J2.57
- net SPI1_MOSI: now also J2.56
- net SPI1_SCK: now also J2.55
- net UART0_CTS: now also J2.43
- net UART0_DCD: now also J2.46
- net UART0_DSR: now also J2.45
- net UART0_RI: now also J2.47
- net UART0_RTS: now also J2.44
- net UART3_RX: now also J2.42
- net UART3_TX: now also J2.41
- net VCC_1V8: now also J2.135, J2.136, J2.186, J2.187; no longer J2.35, J2.36
- net VCC_3V3: now also J2.133, J2.134, J2.185, J2.188; no longer J2.33, J2.34
- net VCC_5V: now also J2.131, J2.132, J2.183, J2.184; no longer J2.31, J2.32
- net VIO_BANK0: now also J2.139, J2.191; no longer J2.39
- net VIO_BANK1: now also J2.140, J2.192; no longer J2.40
- net VIO_BANK2: now also J2.141, J2.193
- net VIO_BANK3: now also J2.142, J2.194
- net VREF_IO: now also J2.137, J2.138, J2.189, J2.190; no longer J2.37, J2.38
- net sMDC: now also J2.116; no longer J2.16
Changed lines of the file:
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@@
 		(lib_id "Connector:SODIMM-200")
 		(at 167.64 147.32 0)
-		(unit 1)
+		(unit 2)
 		(exclude_from_sim no)
 		(in_bom yes)
@@
 				(path "/5d9e1dfb-5ec5-4e06-bbdb-9cbfa1c0b9f1/0260e008-78ae-4c2c-85f8-b31739d2ea08/f6e289d8-1e57-42c9-86d8-5b4c62dbd3c6"
 					(reference "J2")
-					(unit 1)
-				)
-			)
+					(unit 2)
+				)
+			)

Commit message: Iniciado projeto da PCB, para uma referência de tamanho.
Parts:
- J2: footprint (none) -> Connector_PCBEdge:SODIMM-200_2.5V_Card_edge
Changed lines of the file:
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@@
 					(size 1.27 1.27)
 				)
-				(hide yes)
 			)
 		)
@@
 		(on_board yes)
 		(dnp no)
-		(fields_autoplaced yes)
 		(property "Reference" "J2"
 			(at 167.64 41.91 0)
@@
 			)
 		)
-		(property "Footprint" ""
-			(at 203.2 49.53 0)
+		(property "Footprint" "Connector_PCBEdge:SODIMM-200_2.5V_Card_edge"
+			(at 167.64 38.1 0)
 			(effects
 				(font
 					(size 1.27 1.27)
 				)
-				(hide yes)
-			)
-		)
+			)
+		)

Commit message: Adicionado Footprints, criado a visualização da PCB
Connections:
- net GND: now also J1.24
- net MCU_BOOT0: now also J1.27
- net MCU_BOOT1: now also J1.28
- net MCU_EN: now also J1.26
- net MCU_RST_N: now also J1.25
- net VCC_IN: now also J1.23
Changed lines of the file:
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@@
 	(wire
 		(pts
+			(xy 45.72 83.82) (xy 55.88 83.82)
+		)
+		(stroke
+			(width 0)
+			(type default)
+		)
+	)
+	(wire
+		(pts
 			(xy 139.7 55.88) (xy 149.86 55.88)
 		)
@@
 	(wire
 		(pts
+			(xy 91.44 81.28) (xy 101.6 81.28)
+		)
+		(stroke
+			(width 0)
+			(type default)
+		)
+	)
+	(wire
+		(pts
 			(xy 185.42 91.44) (xy 195.58 91.44)
 		)
@@
 	(wire
 		(pts
-			(xy 91.44 86.36) (xy 99.06 86.36)
+			(xy 91.44 86.36) (xy 101.6 86.36)
 		)
 		(stroke
@@
 	(wire
 		(pts
+			(xy 91.44 83.82) (xy 101.6 83.82)
+		)
+		(stroke
+			(width 0)
+			(type default)
+		)
+	)
+	(wire
+		(pts
 			(xy 139.7 162.56) (xy 149.86 162.56)
 		)
@@
 	(wire
 		(pts
+			(xy 45.72 81.28) (xy 55.88 81.28)
+		)
+		(stroke
+			(width 0)
+			(type default)
+		)
+	)
+	(wire
+		(pts
 			(xy 139.7 144.78) (xy 149.86 144.78)
 		)
@@
 	(wire
 		(pts
+			(xy 91.44 78.74) (xy 101.6 78.74)
+		)
+		(stroke
+			(width 0)
+			(type default)
+		)
+	)
+	(wire
+		(pts
 			(xy 185.42 241.3) (xy 195.58 241.3)
 		)
@@
 	(wire
 		(pts
+			(xy 45.72 78.74) (xy 55.88 78.74)
+		)
+		(stroke
+			(width 0)
+			(type default)
+		)
+	)
+	(wire
+		(pts
 			(xy 139.7 218.44) (xy 149.86 218.44)
 		)
@@
 	(wire
 		(pts
-			(xy 91.44 99.06) (xy 99.06 99.06)
+			(xy 91.44 99.06) (xy 101.6 99.06)
 		)
 		(stroke
@@
 	(wire
 		(pts
-			(xy 91.44 88.9) (xy 99.06 88.9)
+			(xy 91.44 88.9) (xy 101.6 88.9)
 		)
 		(stroke
@@
 	(wire
 		(pts
-			(xy 91.44 93.98) (xy 99.06 93.98)
+			(xy 91.44 93.98) (xy 101.6 93.98)
 		)
 		(stroke
@@
 	(wire
 		(pts
-			(xy 91.44 96.52) (xy 99.06 96.52)
+			(xy 91.44 96.52) (xy 101.6 96.52)
 		)
 		(stroke
@@
 	(wire
 		(pts
-			(xy 91.44 91.44) (xy 99.06 91.44)
+			(xy 91.44 91.44) (xy 101.6 91.44)
 		)
 		(stroke
@@
 	(global_label "UART0_RX"
 		(shape passive)
-		(at 99.06 93.98 0)
+		(at 101.6 93.98 0)
 		(effects
 			(font
@@
 		)
 		(property "Intersheetrefs" "${INTERSHEET_REFS}"
-			(at 99.06 93.98 0)
+			(at 101.6 93.98 0)
 			(effects
 				(font
@@
 	(global_label "UART1_RX"
 		(shape passive)
-		(at 99.06 96.52 0)
+		(at 101.6 96.52 0)
 		(effects
 			(font
@@
 		)
 		(property "Intersheetrefs" "${INTERSHEET_REFS}"
-			(at 99.06 96.52 0)
+			(at 101.6 96.52 0)
 			(effects
 				(font
@@
 	(global_label "I2C1_SDA"
 		(shape passive)
-		(at 99.06 88.9 0)
+		(at 101.6 88.9 0)
 		(effects
 			(font
@@
 		)
 		(property "Intersheetrefs" "${INTERSHEET_REFS}"
-			(at 99.06 88.9 0)
+			(at 101.6 88.9 0)
 			(effects
 				(font
@@
 	(global_label "UART2_RX"
 		(shape passive)
-		(at 99.06 99.06 0)
+		(at 101.6 99.06 0)
 		(effects
 			(font
@@
 		)
 		(property "Intersheetrefs" "${INTERSHEET_REFS}"
-			(at 99.06 99.06 0)
+			(at 101.6 99.06 0)
 			(effects
 				(font
@@
 	(global_label "I2C2_SDA"
 		(shape passive)
-		(at 99.06 91.44 0)
+		(at 101.6 91.44 0)
 		(effects
 			(font
@@
 		)
 		(property "Intersheetrefs" "${INTERSHEET_REFS}"
-			(at 99.06 91.44 0)
+			(at 101.6 91.44 0)
 			(effects
 				(font
@@
 	(global_label "I2C0_SDA"
 		(shape passive)
-		(at 99.06 86.36 0)
+		(at 101.6 86.36 0)
 		(effects
 			(font
@@
 		)
 		(property "Intersheetrefs" "${INTERSHEET_REFS}"
-			(at 99.06 86.36 0)
+			(at 101.6 86.36 0)
 			(effects
 				(font
